File: Kicad/boards/26proto.kicad_sch (KiCad schematic)
At the start: 4 parts, among them J1 5051104096, U1 MOUDLE-SEEEDUINO-XIAO-ESP32C3, U2 MOUDLE-SEEEDUINO-XIAO-ESP32C3, U3 MAX3485

Commit message: edited sch
Parts:
- removed U2: MOUDLE-SEEEDUINO-XIAO-ESP32C3, MOUDLE14P-SMD-2.54-21X17.8MM, symbol XIAO_ESP32C3:MOUDLE-SEEEDUINO-XIAO-ESP32C3
- added J2: Micro_SD_Card, symbol Connector:Micro_SD_Card
- added U10: ~, symbol New_Library:Adafruit_DPS310
- added U2, U4, U6: MAX3485, Package_SO:SOIC-8_3.9x4.9mm_P1.27mm, symbol Interface_UART:MAX3485
- added U5, U7: MOUDLE-SEEEDUINO-XIAO-ESP32C3, MOUDLE14P-SMD-2.54-21X17.8MM, symbol Seeed_Studio_XIAO_Series:XIAO-ESP32-C3-SMD
- added U8: ~, symbol New_Library:AS5600
- U1: symbol XIAO_ESP32C3:MOUDLE-SEEEDUINO-XIAO-ESP32C3 -> Seeed_Studio_XIAO_Series:XIAO-ESP32-C3-SMD
Connections:
- net +3.3V: now also U1.12 (3V3), J2.4 (VDD), U10. (VIN), U2.8 (VCC), U4.8 (VCC), U5.12 (3V3), U6.8 (VCC), U8. (OUT)
- net CS: now also U1.1 (GPIO2_A0_D0)
- net DCX-SCLK: now also U1.9 (GPIO8_D8_SCK)
- net GND: now also U1.13 (GND), U1.16 (GND), J2.6 (VSS), J2.9 (SHIELD), U10. (VIN), U2.5 (GND), U4.5 (GND), U5.13 (GND), U5.16 (GND), U6.5 (GND), U8. (OUT)
- net SDA-MOSI: now also U1.11 (GPIO10_D10_MOSI)
- net SDO-MISO: now also U1.10 (GPIO9_D9_MISO)
- net WRX-D/C: now reaches J1.12
- net WRX-D/C: now also U1.2 (GPIO3_A1_D1)
- net at U1.6 (GPIO7_D5_SCL): now also U4.2 (~{RE}), U4.3 (DE)
- net at U1.7 (GPIO21_D6_TX): now also U4.4 (DI)
- net at U1.8 (GPIO20_D7_RX): now also U4.1 (RO)
- new net: U2.1 (RO), U5.8 (GPIO20_D7_RX)
- new net: U2.2 (~{RE}), U2.3 (DE), U5.6 (GPIO7_D5_SCL)
- new net: U2.4 (DI), U5.7 (GPIO21_D6_TX)
- new net: U6.2 (~{RE}), U6.3 (DE)
- new net +BATT: U1.15 (BAT), U5.15 (BAT)
- new net CS_SD: J2.2 (DAT3/CD), U5.1 (GPIO2_A0_D0)
- new net MISO_SD: J2.7 (DAT0), U5.10 (GPIO9_D9_MISO)
- new net MOSI_SD: J2.3 (CMD), U5.11 (GPIO10_D10_MOSI)
- new net RS485_A: U2.6 (A), U4.6 (A), U6.6 (A)
- new net RS485_B: U2.7 (B), U4.7 (B), U6.7 (B)
- new net SCLK_SD: J2.5 (CLK), U5.9 (GPIO8_D8_SCK)
- new net SCL_airdata: U10. (VIN), U8. (OUT)
- new net SDA_aridata: U10. (VIN), U8. (OUT)
- no-connect marks 6 -> 32
Other:
- moved on the sheet: J1, U1, U3

Commit message: edited schimatic
Parts:
- added C1: C_Small, symbol Device:C_Small
Connections:
- net +3.3V: now also C1.1
- net GND: now also C1.2
- no-connect marks 32 -> 31
Changed lines of the file:
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@@
 	(paper "A4")
 	(junction
+		(at 101.6 113.03)
+		(diameter 0)
+		(color 0 0 0 0)
+	)
+	(junction
 		(at 241.3 109.22)
 		(diameter 0)
@@
 	)
 	(junction
+		(at 101.6 118.11)
+		(diameter 0)
+		(color 0 0 0 0)
+	)
+	(junction
 		(at 50.8 71.12)
 		(diameter 0)
@@
 	)
 	(no_connect
-		(at 320.04 114.3)
-	)
-	(no_connect
 		(at 146.05 35.56)
 	)
@@
 	(wire
 		(pts
-			(xy 107.95 113.03) (xy 118.11 113.03)
+			(xy 99.06 113.03) (xy 101.6 113.03)
 		)
 		(stroke
@@
 	(wire
 		(pts
-			(xy 107.95 118.11) (xy 118.11 118.11)
+			(xy 99.06 118.11) (xy 101.6 118.11)
 		)
 		(stroke
@@
 	(wire
 		(pts
+			(xy 101.6 118.11) (xy 118.11 118.11)
+		)
+		(stroke
+			(width 0)
+			(type default)
+		)
+	)
+	(wire
+		(pts
 			(xy 54.61 71.12) (xy 71.12 71.12)
 		)
@@
 	(wire
 		(pts
+			(xy 101.6 113.03) (xy 118.11 113.03)
+		)
+		(stroke
+			(width 0)
+			(type default)
+		)
+	)
+	(wire
+		(pts
 			(xy 215.9 110.49) (xy 234.95 110.49)
 		)
@@
 	)
 	(symbol
+		(lib_id "Device:C_Small")
+		(at 101.6 115.57 0)
+		(unit 1)
+		(exclude_from_sim no)
+		(in_bom yes)
+		(on_board yes)
+		(dnp no)
+		(fields_autoplaced yes)
+		(property "Reference" "C1"
+			(at 104.14 114.3062 0)
+			(effects
+				(font
+					(size 1.27 1.27)
+				)
+				(justify left)
+			)
+		)
+		(property "Value" "C_Small"
+			(at 104.14 116.8462 0)
+			(effects
+				(font
+					(size 1.27 1.27)
+				)
+				(justify left)
+			)
+		)
+		(property "Footprint" ""
+			(at 101.6 115.57 0)
+			(effects
+				(font
+					(size 1.27 1.27)
+				)
+				(hide yes)
+			)
+		)
+		(property "Datasheet" "~"
+			(at 101.6 115.57 0)
+			(effects
+				(font
+					(size 1.27 1.27)
+				)
+				(hide yes)
+			)
+		)
+		(property "Description" "Unpolarized capacitor, small symbol"
+			(at 101.6 115.57 0)
+			(effects
+				(font
+					(size 1.27 1.27)
+				)
+				(hide yes)
+			)
+		)
+		(pin "1"
+		)
+		(pin "2"
+		)
+		(instances
+			(project ""
+				(path "/493bec57-bd9f-4f18-b3ef-0d7a091ad475"
+					(reference "C1")
+					(unit 1)
+				)
+			)
+		)
+	)
+	(symbol
 		(lib_id "power:GND")
 		(at 110.49 35.56 0)
@@
 	(symbol
 		(lib_id "power:GND")
-		(at 107.95 118.11 270)
+		(at 99.06 118.11 270)
 		(mirror x)
 		(unit 1)
@@
 		(dnp no)
 		(property "Reference" "#PWR015"
-			(at 101.6 118.11 0)
+			(at 92.71 118.11 0)
 			(effects
 				(font
@@
 		)
 		(property "Value" "GND"
-			(at 104.394 117.856 0)
+			(at 95.504 117.856 0)
 			(effects
 				(font
@@
 		)
 		(property "Footprint" ""
-			(at 107.95 118.11 0)
+			(at 99.06 118.11 0)
 			(effects
 				(font
@@
 		)
 		(property "Datasheet" ""
-			(at 107.95 118.11 0)
+			(at 99.06 118.11 0)
 			(effects
 				(font
@@
 		)
 		(property "Description" "Power symbol creates a global label with name \"GND\" , ground"
-			(at 107.95 118.11 0)
+			(at 99.06 118.11 0)
 			(effects
 				(font
@@
 	(symbol
 		(lib_id "power:+3.3V")
-		(at 107.95 113.03 90)
+		(at 99.06 113.03 90)
 		(unit 1)
 		(exclude_from_sim no)
@@
 		(fields_autoplaced yes)
 		(property "Reference" "#PWR014"
-			(at 111.76 113.03 0)
+			(at 102.87 113.03 0)
 			(effects
 				(font
@@
 		)
 		(property "Value" "+3.3V"
-			(at 104.14 113.0299 90)
+			(at 95.25 113.0299 90)
 			(effects
 				(font
@@
 		)
 		(property "Footprint" ""
-			(at 107.95 113.03 0)
+			(at 99.06 113.03 0)
 			(effects
 				(font
@@
 		)
 		(property "Datasheet" ""
-			(at 107.95 113.03 0)
+			(at 99.06 113.03 0)
 			(effects
 				(font
@@
 		)
 		(property "Description" "Power symbol creates a global label with name \"+3.3V\""
-			(at 107.95 113.03 0)
+			(at 99.06 113.03 0)
 			(effects
 				(font

Commit message: Update 26proto.kicad_sch
Parts:
- removed U3: MAX3485, Package_SO:SOIC-8_3.9x4.9mm_P1.27mm, symbol Interface_UART:MAX3485
- added J3, J4: Conn_01x04, symbol Connector_Generic:Conn_01x04
- added R1, R2, R3: R, symbol Device:R
- added RV1, RV2, RV3: R_Potentiometer, symbol Device:R_Potentiometer
- added U11: MOUDLE-SEEEDUINO-XIAO-ESP32C3, MOUDLE14P-SMD-2.54-21X17.8MM, symbol Seeed_Studio_XIAO_Series:XIAO-ESP32-C3-SMD
- added U9: MAX3485, Package_SO:SOIC-8_3.9x4.9mm_P1.27mm, symbol Interface_UART:MAX3485
Connections:
- net +3.3V: now also U7.12 (3V3), J3.1 (Pin_1), J4.1 (Pin_1), R1.2, R2.2, R3.2, RV1.3, RV2.3, RV3.3, U11.12 (3V3), U9.8 (VCC)
- net +BATT: now also U7.15 (BAT), U11.15 (BAT)
- net CS_SD: now also R2.1
- net Encoder_Apin: now also U7.10 (GPIO9_D9_MISO), J4.3 (Pin_3)
- net Encoder_Bpin: now also U7.9 (GPIO8_D8_SCK), J4.4 (Pin_4)
- net GND: now also U7.13 (GND), U7.16 (GND), J3.2 (Pin_2), J4.2 (Pin_2), RV1.1, RV2.1, RV3.1, U11.13 (GND), U11.16 (GND), U9.5 (GND)
- net MISO_SD: now also R3.1
- net MOSI_SD: now also R1.1
- net Pot_elv: now also RV1.2, U11.1 (GPIO2_A0_D0)
- net Pot_rud: now also RV2.2, U11.2 (GPIO3_A1_D1)
- net Pot_trim: now also RV3.2, U11.3 (GPIO4_A2_D2)
- net RS485_A: now also U9.6 (A)
- net RS485_B: now also U9.7 (B)
- net SCL_airdata: now also U7.6 (GPIO7_D5_SCL)
- net SDA_airdata: now also U7.5 (GPIO6_D4_SDA)
- net at U2.2 (~{RE}), U2.3 (DE): now also U5.4 (GPIO5_A3_D3); no longer U5.6 (GPIO7_D5_SCL)
- net at U4.2 (~{RE}), U4.3 (DE): now also U1.4 (GPIO5_A3_D3); no longer U1.6 (GPIO7_D5_SCL)
- net SDA_BNO085: now reaches U5.5 (GPIO6_D4_SDA)
- net at U6.1 (RO): now also U7.8 (GPIO20_D7_RX)
- net at U6.2 (~{RE}), U6.3 (DE): now also U7.11 (GPIO10_D10_MOSI)
- net at U6.4 (DI): now also U7.7 (GPIO21_D6_TX)
- net SDA_board3: now reaches U1.5 (GPIO6_D4_SDA)
- net SDA_board3: now also U11.5 (GPIO6_D4_SDA)
- new net: U11.8 (GPIO20_D7_RX), U9.1 (RO)
- new net: U11.11 (GPIO10_D10_MOSI), U9.2 (~{RE}), U9.3 (DE)
- new net: U11.7 (GPIO21_D6_TX), U9.4 (DI)
- new net RX_URM37: J3.3 (Pin_3), U11.10 (GPIO9_D9_MISO)
- new net SCL_BNO085: U5.6 (GPIO7_D5_SCL)
- new net SCL_board3: U1.6 (GPIO7_D5_SCL), U11.6 (GPIO7_D5_SCL)
- new net TX_URM37: J3.4 (Pin_4), U11.9 (GPIO8_D8_SCK)
- no-connect marks 31 -> 66
Other:
- moved on the sheet: C1, J1, J2, U1, U10, U2, U4, U5, U6, U7, U8

Commit message: upgraded schema
Connections:
- net RES: now also U1.3 (GPIO4_A2_D2)
- no-connect marks 66 -> 65
Other:
- moved on the sheet: J1, RV1, RV2, RV3, U11, U9

Commit message: updated sch
Parts:
- removed U9: MAX3485, Package_SO:SOIC-8_3.9x4.9mm_P1.27mm, symbol Interface_UART:MAX3485
- added J5, J6, J7, J8, J9: Conn_01x04, Connector_JST:JST_XH_S4B-XH-SM4-TB_1x04-1MP_P2.50mm_Horizontal, symbol Connector_Generic:Conn_01x04
- added R4, R5: R, Resistor_SMD:R_0201_0603Metric_Pad0.64x0.40mm_HandSolder, symbol Device:R
- C1: footprint (none) -> Capacitor_SMD:C_0201_0603Metric_Pad0.64x0.40mm_HandSolder
- J1: footprint 5051104096:CON_5051104096_MOL -> footprints:CON_5051104096_MOL
- J2: footprint (none) -> Connector_Card:microSD_HC_Hirose_DM3AT-SF-PEJM5
- J3, J4: footprint (none) -> Connector_JST:JST_XH_B4B-XH-A_1x04_P2.50mm_Vertical
- R1, R2, R3: footprint (none) -> Resistor_SMD:R_0201_0603Metric_Pad0.64x0.40mm_HandSolder
- RV1, RV2, RV3: footprint (none) -> Connector_JST:JST_XH_B3B-XH-A_1x03_P2.50mm_Vertical
- U1, U11, U5, U7: footprint MOUDLE14P-SMD-2.54-21X17.8MM -> footprints:XIAO-ESP32C3-SMD
- U10: value ~ -> Adafruit DPS310; footprint (none) -> Connector_JST:JST_XH_B7B-XH-A_1x07_P2.50mm_Vertical
- U8: value ~ -> AS5600 breakout board; footprint (none) -> Connector_JST:JST_XH_B6B-XH-A_1x06_P2.50mm_Vertical
Connections:
- net +3.3V: now also U10.2 (3Vo), U10.7 (CS), U8.2 (3V3), J9.1 (Pin_1); no longer U10. (VIN), U8. (OUT)
- net GND: now also U10.3 (GND), U10.5 (SDO), U8.3 (GND), J5.2 (Pin_2), J6.2 (Pin_2), J7.2 (Pin_2), J8.2 (Pin_2), J9.2 (Pin_2); no longer U10. (VIN), U8. (OUT)
- net RS485_A: now also J5.3 (Pin_3), J6.3 (Pin_3), J7.3 (Pin_3), J8.3 (Pin_3), R4.2, R5.2
- net RS485_B: now also J5.4 (Pin_4), J6.4 (Pin_4), J7.4 (Pin_4), J8.4 (Pin_4), R4.1, R5.1
- net SCL_BNO085: now also J9.4 (Pin_4)
- net SCL_airdata: now also U10.4 (SCK), U8.4 (SCL); no longer U10. (VIN), U8. (OUT)
- net SDA_BNO085: now also J9.3 (Pin_3)
- net SDA_aridata: now also U10.6 (SDI), U8.5 (SDA); no longer U10. (VIN), U8. (OUT)
- no-connect marks 65 -> 72
Other:
- moved on the sheet: J3, RV1, RV2, RV3, U6, U7

Commit message: edited pcb
Parts:
- AS5600: renamed from U8; footprint Connector_JST:JST_XH_B6B-XH-A_1x06_P2.50mm_Vertical -> Connector_PinHeader_2.54mm:PinHeader_1x06_P2.54mm_Vertical
- DPS310: renamed from U10; footprint Connector_JST:JST_XH_B7B-XH-A_1x07_P2.50mm_Vertical -> Connector_PinHeader_2.54mm:PinHeader_1x07_P2.54mm_Vertical
- J3: value Conn_01x04 -> URM37; footprint Connector_JST:JST_XH_B4B-XH-A_1x04_P2.50mm_Vertical -> Connector_JST:JST_XH_S4B-XH-SM4-TB_1x04-1MP_P2.50mm_Horizontal
- J4: value Conn_01x04 -> RE12A; footprint Connector_JST:JST_XH_B4B-XH-A_1x04_P2.50mm_Vertical -> Connector_JST:JST_XH_S4B-XH-SM4-TB_1x04-1MP_P2.50mm_Horizontal
- J5: value Conn_01x04 -> RS485_TFT
- J6: value Conn_01x04 -> RS485_airdata
- J7: value Conn_01x04 -> RS485_logger_2
- J8: value Conn_01x04 -> RS485_logger
- J9: value Conn_01x04 -> BNO085; footprint Connector_JST:JST_XH_S4B-XH-SM4-TB_1x04-1MP_P2.50mm_Horizontal -> footprints:MODULE_4754
- RV1, RV2, RV3: footprint Connector_JST:JST_XH_B3B-XH-A_1x03_P2.50mm_Vertical -> Connector_JST:JST_XH_S3B-XH-SM4-TB_1x03-1MP_P2.50mm_Horizontal
- U1: value MOUDLE-SEEEDUINO-XIAO-ESP32C3 -> MOUDLE-SEEEDUINO-XIAO-ESP32C3_TFT
- U11: value MOUDLE-SEEEDUINO-XIAO-ESP32C3 -> MOUDLE-SEEEDUINO-XIAO-ESP32C3_pot
- U5: value MOUDLE-SEEEDUINO-XIAO-ESP32C3 -> MOUDLE-SEEEDUINO-XIAO-ESP32C3_logger
- U7: value MOUDLE-SEEEDUINO-XIAO-ESP32C3 -> MOUDLE-SEEEDUINO-XIAO-ESP32C3_airdata
Changed lines of the file:
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@@
 			)
 		)
-		(property "Footprint" "Connector_JST:JST_XH_B3B-XH-A_1x03_P2.50mm_Vertical"
+		(property "Footprint" "Connector_JST:JST_XH_S3B-XH-SM4-TB_1x03-1MP_P2.50mm_Horizontal"
 			(at 311.15 85.09 0)
 			(effects
@@
 			)
 		)
-		(property "Value" "Conn_01x04"
+		(property "Value" "BNO085"
 			(at 119.38 189.2299 0)
 			(effects
@@
 			)
 		)
-		(property "Footprint" "Connector_JST:JST_XH_S4B-XH-SM4-TB_1x04-1MP_P2.50mm_Horizontal"
+		(property "Footprint" "footprints:MODULE_4754"
 			(at 116.84 186.69 0)
 			(effects
@@
 			)
 		)
-		(property "Value" "MOUDLE-SEEEDUINO-XIAO-ESP32C3"
+		(property "Value" "MOUDLE-SEEEDUINO-XIAO-ESP32C3_pot"
 			(at 282.194 20.32 0)
 			(effects
@@
 			)
 		)
-		(property "Footprint" "Connector_JST:JST_XH_B3B-XH-A_1x03_P2.50mm_Vertical"
+		(property "Footprint" "Connector_JST:JST_XH_S3B-XH-SM4-TB_1x03-1MP_P2.50mm_Horizontal"
 			(at 285.75 85.09 0)
 			(effects
@@
 			)
 		)
-		(property "Value" "Conn_01x04"
+		(property "Value" "RS485_airdata"
 			(at 299.72 209.5499 0)
 			(effects
@@
 			)
 		)
-		(property "Value" "Conn_01x04"
+		(property "Value" "RE12A"
 			(at 299.72 195.5799 0)
 			(effects
@@
 			)
 		)
-		(property "Footprint" "Connector_JST:JST_XH_B4B-XH-A_1x04_P2.50mm_Vertical"
+		(property "Footprint" "Connector_JST:JST_XH_S4B-XH-SM4-TB_1x04-1MP_P2.50mm_Horizontal"
 			(at 297.18 193.04 0)
 			(effects
@@
 		(dnp no)
 		(fields_autoplaced yes)
-		(property "Reference" "U10"
-			(at 384.556 235.712 90)
+		(property "Reference" "DPS310"
+			(at 389.89 219.7099 90)
 			(effects
 				(font
@@
 		)
 		(property "Value" "Adafruit DPS310"
-			(at 377.698 233.172 90)
+			(at 389.89 222.2499 90)
 			(effects
 				(font
@@
 			)
 		)
-		(property "Footprint" "Connector_JST:JST_XH_B7B-XH-A_1x07_P2.50mm_Vertical"
+		(property "Footprint" "Connector_PinHeader_2.54mm:PinHeader_1x07_P2.54mm_Vertical"
 			(at 389.89 218.44 0)
 			(effects
@@
 			(project ""
 				(path "/493bec57-bd9f-4f18-b3ef-0d7a091ad475"
-					(reference "U10")
+					(reference "DPS310")
 					(unit 1)
 				)
@@
 			)
 		)
-		(property "Value" "MOUDLE-SEEEDUINO-XIAO-ESP32C3"
+		(property "Value" "MOUDLE-SEEEDUINO-XIAO-ESP32C3_logger"
 			(at 41.148 192.532 0)
 			(effects
@@
 			)
 		)
-		(property "Value" "Conn_01x04"
+		(property "Value" "RS485_TFT"
 			(at 72.39 114.2999 0)
 			(effects
@@
 			)
 		)
-		(property "Value" "Conn_01x04"
+		(property "Value" "RS485_logger_2"
 			(at 119.38 201.9299 0)
 			(effects
@@
 			)
 		)
-		(property "Value" "Conn_01x04"
+		(property "Value" "URM37"
 			(at 35.56 115.5699 0)
 			(effects
@@
 			)
 		)
-		(property "Footprint" "Connector_JST:JST_XH_B4B-XH-A_1x04_P2.50mm_Vertical"
+		(property "Footprint" "Connector_JST:JST_XH_S4B-XH-SM4-TB_1x04-1MP_P2.50mm_Horizontal"
 			(at 33.02 113.03 0)
 			(effects
@@
 			)
 		)
-		(property "Value" "MOUDLE-SEEEDUINO-XIAO-ESP32C3"
+		(property "Value" "MOUDLE-SEEEDUINO-XIAO-ESP32C3_airdata"
 			(at 341.122 112.268 0)
 			(effects
@@
 		(on_board yes)
 		(dnp no)
-		(property "Reference" "U8"
+		(property "Reference" "AS5600"
 			(at 355.6 222.2499 90)
 			(effects
@@
 			)
 		)
-		(property "Footprint" "Connector_JST:JST_XH_B6B-XH-A_1x06_P2.50mm_Vertical"
+		(property "Footprint" "Connector_PinHeader_2.54mm:PinHeader_1x06_P2.54mm_Vertical"
 			(at 345.44 223.52 0)
 			(effects
@@
 			(project ""
 				(path "/493bec57-bd9f-4f18-b3ef-0d7a091ad475"
-					(reference "U8")
+					(reference "AS5600")
 					(unit 1)
 				)
@@
 			)
 		)
-		(property "Value" "MOUDLE-SEEEDUINO-XIAO-ESP32C3"
+		(property "Value" "MOUDLE-SEEEDUINO-XIAO-ESP32C3_TFT"
 			(at 19.812 14.478 0)
 			(effects
@@
 			)
 		)
-		(property "Footprint" "Connector_JST:JST_XH_B3B-XH-A_1x03_P2.50mm_Vertical"
+		(property "Footprint" "Connector_JST:JST_XH_S3B-XH-SM4-TB_1x03-1MP_P2.50mm_Horizontal"
 			(at 262.89 85.09 0)
 			(effects
@@
 			)
 		)
-		(property "Value" "Conn_01x04"
+		(property "Value" "RS485_logger"
 			(at 119.38 215.8999 0)
 			(effects

Commit message: edited sch and pcb
Parts:
- added Q2: NPN, Package_TO_SOT_SMD:SOT-23, symbol Simulation_SPICE:NPN
- added R6, R7, R8: R, Resistor_SMD:R_0201_0603Metric_Pad0.64x0.40mm_HandSolder, symbol Device:R
Connections:
- net +3.3V: now also R6.1; no longer J4.1 (Pin_1)
- net GND: now also J4.3 (Pin_3), J4.4 (Pin_4); no longer J4.2 (Pin_2)
- net Encoder_Apin renamed encoder_out
- net encoder_out: now also Q2.3 (E); no longer J4.3 (Pin_3)
- net Encoder_Bpin: no longer names the net of U7.9 (GPIO8_D8_SCK)
- net Encoder_Bpin: no longer J4.4 (Pin_4)
- new net: Q2.1 (C), R6.2
- new net: J4.1 (Pin_1), R7.2
- new net +5V: R7.1, R8.1
- new net encoder_raw: J4.2 (Pin_2), Q2.2 (B), R8.2
- no-connect marks 72 -> 73
