File: Kicad/boards/26proto.kicad_sch (KiCad schematic)
At the start: 39 parts, among them J1 5051104096, J10 Conn_01x05, J2 Micro_SD_Card, J3 URM37, J4 RE12A, J5 RS485_TFT, J6 RS485_airdata, J7 RS485_logger_2, J8 RS485_logger, J9 BNO085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

Commit message: edited pcb
Parts:
- added R15, R16: R, Resistor_SMD:R_0201_0603Metric_Pad0.64x0.40mm_HandSolder, symbol Device:R
- Q2: symbol Simulation_SPICE:NPN -> Transistor_BJT:MMBT2222A
Connections:
- net SDA_aridata is gone; now on net SDA_airdata: AS5600.5 (SDA), AS5601.5 (SDA), DPS310.6 (SDI)
- net +5V: now also U7.14 (5V)
- net GND: now also R15.1; no longer Q2.3 (E), R14.2
- net encoder_out: now also Q2.3 (C); no longer Q2.1 (C)
- net encoder_raw: now also R16.2; no longer J4.2 (Pin_2), R8.2
- new net: J4.2 (Pin_2), R16.1, R8.2
- new net: Q2.1 (B), R14.2, R15.2
- no-connect marks 84 -> 83
Changed lines of the file:
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@@
 	)
 	(junction
-		(at 288.29 146.05)
-		(diameter 0)
-		(color 0 0 0 0)
-	)
-	(junction
 		(at 358.14 175.26)
 		(diameter 0)
@@
 	)
 	(junction
+		(at 288.29 146.05)
+		(diameter 0)
+		(color 0 0 0 0)
+	)
+	(junction
 		(at 204.47 77.47)
 		(diameter 0)
@@
 	)
 	(no_connect
-		(at 378.46 130.81)
-	)
-	(no_connect
 		(at 198.12 25.4)
 	)
@@
 	(wire
 		(pts
-			(xy 269.24 186.69) (xy 281.94 186.69)
+			(xy 269.24 186.69) (xy 271.78 186.69)
 		)
 		(stroke
@@
 	(wire
 		(pts
+			(xy 279.4 186.69) (xy 281.94 186.69)
+		)
+		(stroke
+			(width 0)
+			(type default)
+		)
+	)
+	(wire
+		(pts
 			(xy 54.61 233.68) (xy 69.85 233.68)
 		)
@@
 	(wire
 		(pts
-			(xy 288.29 146.05) (xy 288.29 151.13)
-		)
-		(stroke
-			(width 0)
-			(type default)
-		)
-	)
-	(wire
-		(pts
 			(xy 76.2 233.68) (xy 77.47 233.68)
 		)
@@
 		)
 	)
-	(global_label "SDA_aridata"
+	(global_label "SDA_airdata"
 		(shape input)
 		(at 336.55 217.17 180)
@@
 		)
 	)
-	(global_label "SDA_aridata"
+	(global_label "SDA_airdata"
 		(shape input)
 		(at 378.46 226.06 180)
@@
 		)
 	)
-	(global_label "SDA_aridata"
+	(global_label "SDA_airdata"
 		(shape input)
 		(at 336.55 240.03 180)
@@
 	)
 	(symbol
+		(lib_id "power:+5V")
+		(at 378.46 130.81 270)
+		(unit 1)
+		(exclude_from_sim no)
+		(in_bom yes)
+		(on_board yes)
+		(dnp no)
+		(fields_autoplaced yes)
+		(property "Reference" "#PWR059"
+			(at 374.65 130.81 0)
+			(effects
+				(font
+					(size 1.27 1.27)
+				)
+				(hide yes)
+			)
+		)
+		(property "Value" "+5V"
+			(at 382.27 130.8099 90)
+			(effects
+				(font
+					(size 1.27 1.27)
+				)
+				(justify left)
+			)
+		)
+		(property "Footprint" ""
+			(at 378.46 130.81 0)
+			(effects
+				(font
+					(size 1.27 1.27)
+				)
+				(hide yes)
+			)
+		)
+		(property "Datasheet" ""
+			(at 378.46 130.81 0)
+			(effects
+				(font
+					(size 1.27 1.27)
+				)
+				(hide yes)
+			)
+		)
+		(property "Description" "Power symbol creates a global label with name \"+5V\""
+			(at 378.46 130.81 0)
+			(effects
+				(font
+					(size 1.27 1.27)
+				)
+				(hide yes)
+			)
+		)
+		(pin "1"
+		)
+		(instances
+			(project ""
+				(path "/493bec57-bd9f-4f18-b3ef-0d7a091ad475"
+					(reference "#PWR059")
+					(unit 1)
+				)
+			)
+		)
+	)
+	(symbol
 		(lib_id "power:GND")
 		(at 292.1 207.01 270)
@@
 	)
 	(symbol
+		(lib_id "Device:R")
+		(at 288.29 149.86 180)
+		(unit 1)
+		(exclude_from_sim no)
+		(in_bom yes)
+		(on_board yes)
+		(dnp no)
+		(property "Reference" "R15"
+			(at 288.544 150.114 90)
+			(effects
+				(font
+					(size 1.27 1.27)
+				)
+			)
+		)
+		(property "Value" "R"
+			(at 289.56 152.908 90)
+			(effects
+				(font
+					(size 1.27 1.27)
+				)
+				(hide yes)
+			)
+		)
+		(property "Footprint" "Resistor_SMD:R_0201_0603Metric_Pad0.64x0.40mm_HandSolder"
+			(at 290.068 149.86 90)
+			(effects
+				(font
+					(size 1.27 1.27)
+				)
+				(hide yes)
+			)
+		)
+		(property "Datasheet" "~"
+			(at 288.29 149.86 0)
+			(effects
+				(font
+					(size 1.27 1.27)
+				)
+				(hide yes)
+			)
+		)
+		(property "Description" "Resistor"
+			(at 288.29 149.86 0)
+			(effects
+				(font
+					(size 1.27 1.27)
+				)
+				(hide yes)
+			)
+		)
+		(pin "1"
+		)
+		(pin "2"
+		)
+		(instances
+			(project "26proto"
+				(path "/493bec57-bd9f-4f18-b3ef-0d7a091ad475"
+					(reference "R15")
+					(unit 1)
+				)
+			)
+		)
+	)
+	(symbol
 		(lib_id "Connector_Generic:Conn_01x02")
 		(at 297.18 220.98 0)
@@
 	)
 	(symbol
+		(lib_id "Device:R")
+		(at 275.59 186.69 270)
+		(mirror x)
+		(unit 1)
+		(exclude_from_sim no)
+		(in_bom yes)
+		(on_board yes)
+		(dnp no)
+		(property "Reference" "R16"
+			(at 275.59 186.436 90)
+			(effects
+				(font
+					(size 1.27 1.27)
+				)
+			)
+		)
+		(property "Value" "R"
+			(at 278.638 187.96 90)
+			(effects
+				(font
+					(size 1.27 1.27)
+				)
+				(hide yes)
+			)
+		)
+		(property "Footprint" "Resistor_SMD:R_0201_0603Metric_Pad0.64x0.40mm_HandSolder"
+			(at 275.59 188.468 90)
+			(effects
+				(font
+					(size 1.27 1.27)
+				)
+				(hide yes)
+			)
+		)
+		(property "Datasheet" "~"
+			(at 275.59 186.69 0)
+			(effects
+				(font
+					(size 1.27 1.27)
+				)
+				(hide yes)
+			)
+		)
+		(property "Description" "Resistor"
+			(at 275.59 186.69 0)
+			(effects
+				(font
+					(size 1.27 1.27)
+				)
+				(hide yes)
+			)
+		)
+		(pin "1"
+		)
+		(pin "2"
+		)
+		(instances
+			(project "26proto"
+				(path "/493bec57-bd9f-4f18-b3ef-0d7a091ad475"
+					(reference "R16")
+					(unit 1)
+				)
+			)
+		)
+	)
+	(symbol
 		(lib_id "power:+3.3V")
 		(at 325.12 247.65 90)
@@
 	(symbol
 		(lib_id "power:GND")
-		(at 288.29 151.13 0)
+		(at 288.29 153.67 0)
 		(unit 1)
 		(exclude_from_sim no)
@@
 		(dnp no)
 		(property "Reference" "#PWR057"
-			(at 288.29 157.48 0)
+			(at 288.29 160.02 0)
 			(effects
 				(font
@@
 		)
 		(property "Value" "GND"
-			(at 288.29 156.21 90)
+			(at 288.29 158.75 90)
 			(effects
 				(font
@@
 		)
 		(property "Footprint" ""
-			(at 288.29 151.13 0)
+			(at 288.29 153.67 0)
 			(effects
 				(font
@@
 		)
 		(property "Datasheet" ""
-			(at 288.29 151.13 0)
+			(at 288.29 153.67 0)
 			(effects
 				(font
@@
 		)
 		(property "Description" "Power symbol creates a global label with name \"GND\" , ground"
-			(at 288.29 151.13 0)
+			(at 288.29 153.67 0)
 			(effects
 				(font
@@
 	)
 	(symbol
-		(lib_id "Simulation_SPICE:NPN")
+		(lib_id "Transistor_BJT:MMBT2222A")
 		(at 293.37 146.05 0)
 		(unit 1)
@@
 		)
 		(property "Footprint" "Package_TO_SOT_SMD:SOT-23"
-			(at 356.87 146.05 0)
+			(at 298.45 147.955 0)
 			(effects
 				(font
 					(size 1.27 1.27)
+					(italic yes)
 				)
+				(justify left)
 				(hide yes)
 			)
 		)
-		(property "Datasheet" "https://ngspice.sourceforge.io/docs/ngspice-html-manual/manual.xhtml#cha_BJTs"
-			(at 356.87 146.05 0)
+		(property "Datasheet" "https://assets.nexperia.com/documents/data-sheet/MMBT2222A.pdf"
+			(at 293.37 146.05 0)
 			(effects
 				(font
 					(size 1.27 1.27)
 				)
+				(justify left)
 				(hide yes)
 			)
 		)
-		(property "Description" "Bipolar transistor symbol for simulation only, substrate tied to the emitter"
+		(property "Description" "600mA Ic, 40V Vce, NPN Transistor, SOT-23"
 			(at 293.37 146.05 0)
 			(effects

Commit message: conflict?
Parts:
- C1: footprint Capacitor_SMD:C_0201_0603Metric_Pad0.64x0.40mm_HandSolder -> Capacitor_SMD:C_0603_1608Metric_Pad1.08x0.95mm_HandSolder
- R1, R10, R11, R12, R13, R14, R15, R16, R2, R3, R4, R5, R6, R7, R8, R9: footprint Resistor_SMD:R_0201_0603Metric_Pad0.64x0.40mm_HandSolder -> Resistor_SMD:R_0603_1608Metric_Pad0.98x0.95mm_HandSolder
Changed lines of the file:
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@@
 			)
 		)
-		(property "Footprint" "Resistor_SMD:R_0201_0603Metric_Pad0.64x0.40mm_HandSolder"
+		(property "Footprint" "Resistor_SMD:R_0603_1608Metric_Pad0.98x0.95mm_HandSolder"
 			(at 294.132 134.62 90)
 			(effects
@@
 			)
 		)
-		(property "Footprint" "Capacitor_SMD:C_0201_0603Metric_Pad0.64x0.40mm_HandSolder"
+		(property "Footprint" "Capacitor_SMD:C_0603_1608Metric_Pad1.08x0.95mm_HandSolder"
 			(at 120.65 236.22 0)
 			(effects
@@
 			)
 		)
-		(property "Footprint" "Resistor_SMD:R_0201_0603Metric_Pad0.64x0.40mm_HandSolder"
+		(property "Footprint" "Resistor_SMD:R_0603_1608Metric_Pad0.98x0.95mm_HandSolder"
 			(at 121.92 239.522 90)
 			(effects
@@
 			)
 		)
-		(property "Footprint" "Resistor_SMD:R_0201_0603Metric_Pad0.64x0.40mm_HandSolder"
+		(property "Footprint" "Resistor_SMD:R_0603_1608Metric_Pad0.98x0.95mm_HandSolder"
 			(at 121.92 229.362 90)
 			(effects
@@
 			)
 		)
-		(property "Footprint" "Resistor_SMD:R_0201_0603Metric_Pad0.64x0.40mm_HandSolder"
+		(property "Footprint" "Resistor_SMD:R_0603_1608Metric_Pad0.98x0.95mm_HandSolder"
 			(at 121.92 226.822 90)
 			(effects
@@
 			)
 		)
-		(property "Footprint" "Resistor_SMD:R_0201_0603Metric_Pad0.64x0.40mm_HandSolder"
+		(property "Footprint" "Resistor_SMD:R_0603_1608Metric_Pad0.98x0.95mm_HandSolder"
 			(at 83.058 46.99 90)
 			(effects
@@
 			)
 		)
-		(property "Footprint" "Resistor_SMD:R_0201_0603Metric_Pad0.64x0.40mm_HandSolder"
+		(property "Footprint" "Resistor_SMD:R_0603_1608Metric_Pad0.98x0.95mm_HandSolder"
 			(at 200.152 102.87 90)
 			(effects
@@
 			)
 		)
-		(property "Footprint" "Resistor_SMD:R_0201_0603Metric_Pad0.64x0.40mm_HandSolder"
+		(property "Footprint" "Resistor_SMD:R_0603_1608Metric_Pad0.98x0.95mm_HandSolder"
 			(at 141.732 83.82 90)
 			(effects
@@
 			)
 		)
-		(property "Footprint" "Resistor_SMD:R_0201_0603Metric_Pad0.64x0.40mm_HandSolder"
+		(property "Footprint" "Resistor_SMD:R_0603_1608Metric_Pad0.98x0.95mm_HandSolder"
 			(at 145.288 93.98 90)
 			(effects
@@
 			)
 		)
-		(property "Footprint" "Resistor_SMD:R_0201_0603Metric_Pad0.64x0.40mm_HandSolder"
+		(property "Footprint" "Resistor_SMD:R_0603_1608Metric_Pad0.98x0.95mm_HandSolder"
 			(at 284.48 147.828 90)
 			(effects
@@
 			)
 		)
-		(property "Footprint" "Resistor_SMD:R_0201_0603Metric_Pad0.64x0.40mm_HandSolder"
+		(property "Footprint" "Resistor_SMD:R_0603_1608Metric_Pad0.98x0.95mm_HandSolder"
 			(at 353.822 203.2 90)
 			(effects
@@
 			)
 		)
-		(property "Footprint" "Resistor_SMD:R_0201_0603Metric_Pad0.64x0.40mm_HandSolder"
+		(property "Footprint" "Resistor_SMD:R_0603_1608Metric_Pad0.98x0.95mm_HandSolder"
 			(at 290.068 149.86 90)
 			(effects
@@
 			)
 		)
-		(property "Footprint" "Resistor_SMD:R_0201_0603Metric_Pad0.64x0.40mm_HandSolder"
+		(property "Footprint" "Resistor_SMD:R_0603_1608Metric_Pad0.98x0.95mm_HandSolder"
 			(at 275.59 188.468 90)
 			(effects
@@
 			)
 		)
-		(property "Footprint" "Resistor_SMD:R_0201_0603Metric_Pad0.64x0.40mm_HandSolder"
+		(property "Footprint" "Resistor_SMD:R_0603_1608Metric_Pad0.98x0.95mm_HandSolder"
 			(at 84.582 46.99 90)
 			(effects
@@
 			)
 		)
-		(property "Footprint" "Resistor_SMD:R_0201_0603Metric_Pad0.64x0.40mm_HandSolder"
+		(property "Footprint" "Resistor_SMD:R_0603_1608Metric_Pad0.98x0.95mm_HandSolder"
 			(at 275.59 194.818 90)
 			(effects
@@
 			)
 		)
-		(property "Footprint" "Resistor_SMD:R_0201_0603Metric_Pad0.64x0.40mm_HandSolder"
+		(property "Footprint" "Resistor_SMD:R_0603_1608Metric_Pad0.98x0.95mm_HandSolder"
 			(at 132.08 249.682 90)
 			(effects
@@
 			)
 		)
-		(property "Footprint" "Resistor_SMD:R_0201_0603Metric_Pad0.64x0.40mm_HandSolder"
+		(property "Footprint" "Resistor_SMD:R_0603_1608Metric_Pad0.98x0.95mm_HandSolder"
 			(at 275.59 192.278 90)
 			(effects

Commit message: added mosfet
Parts:
- added BT1: Battery_Cell, Battery:BatteryHolder_Seiko_MS621F, symbol Device:Battery_Cell
- added Q1: 2N7000, Package_TO_SOT_THT:TO-92_Inline, symbol Transistor_FET:2N7000
- added U3: 1339D, Package_SO:TSSOP-8_3x3mm_P0.65mm, symbol New_Library:1339D
- added Y1: CFS-206, Crystal:Crystal_DS26_D2.0mm_L6.0mm_Vertical, symbol Device:Crystal
- J9: footprint 4754:MODULE_4754 -> footprints:MODULE_4754_without_holes
Connections:
- net +3.3V: now also U3. (Vcc)
- net GND: now also BT1.2 (-), U3. (Vcc)
- net SCL_board3: now also U3.6 (SCL)
- net SDA_board3: now also U3.8 (SDA)
- new net: U3.1 (X1), Y1.1
- new net: U3.2 (X2), Y1.2
- new net: BT1.1 (+), U3.3 (V_backup)
- no-connect marks 83 -> 84

Commit message: added RTC
Parts:
- removed Q1: 2N7000, Package_TO_SOT_THT:TO-92_Inline, symbol Transistor_FET:2N7000
- added R17: R, Resistor_THT:R_Axial_DIN0207_L6.3mm_D2.5mm_P7.62mm_Horizontal, symbol Device:R
- added SW1: SW_DIP_x01, footprints:CLSB12A02T, symbol Switch:SW_DIP_x01
Connections:
- net +3.3V: now also U3.8 (Vcc), R17.1; no longer U3. (Vcc)
- net GND: now also U3.4 (GND); no longer J1.34, J1.35, J1.36, J1.37, U3. (Vcc)
- net SDA_board3: now also U3.5 (SDA); no longer U3.8 (SDA)
- net at J1.38: now also SW1.1
- new net: R17.2, SW1.2
- new net MOSFET_source: J1.34, J1.35, J1.36, J1.37
- no-connect marks 84 -> 83
