File: Kicad/boards/TFTboard.kicad_sch (KiCad schematic)
At the start: 24 parts, among them J1 5051104096, J10 Conn_01x04, J13 Conn_01x03 speaker, J3 URM37, J4 Conn_01x03 servo, J5 RS485_TFT, J6 Conn_01x03 encoder_direct, SW1 SW_DIP_x01, U1 MOUDLE-SEEEDUINO-XIAO-ESP32C3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, U11 MOUDLE-SEEEDUINO-XIAO-ESP32C3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

Commit message: 一旦完成
Parts:
- added C3: 47uF, Capacitor_SMD:C_0603_1608Metric_Pad1.08x0.95mm_HandSolder, symbol Device:C_Small
Connections:
- net +3.3V-3: now also C3.1
- net +BATT renamed +BATT-3
- net +BATT-3: no longer U1.15 (BAT)
- net GND renamed GND-3
- net GND-3: now also C3.2
- no-connect marks 41 -> 42

Commit message: edited boards
Parts:
- added R24, R28: 220k, Resistor_SMD:R_0603_1608Metric_Pad0.98x0.95mm_HandSolder, symbol Device:R
Connections:
- net +BATT-3: now also R24.1
- net GND-3: now also R28.2
- net Pot_trim renamed V_check-3
- net V_check-3: now also R24.2, R28.1
Other:
- moved on the sheet: D1, R11, R12, R23, U11
