File: Kicad/boards/loggerboard.kicad_sch (KiCad schematic)
At the start: 21 parts, among them J2 Micro_SD_Card, J7 RS485_logger_2, J8 RS485_logger, J9 BNO085, U2 MAX3485, U5 MOUDLE-SEEEDUINO-XIAO-ESP32C3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, U6 DS3231MZ

Commit message: edited boards
Parts:
- added R33, R34: 220k, Resistor_SMD:R_0603_1608Metric_Pad0.98x0.95mm_HandSolder, symbol Device:R
Connections:
- net +BATT-2: now also R33.1
- net GND-2: now also R34.2
- net V_check-2: now reaches U5.1 (GPIO2_A0_D0)
- net V_check-2: now also R33.2, R34.1
- no-connect marks 23 -> 22
