File: Kicad/boards/untitled.kicad_sch (KiCad schematic)
At the start: 18 parts, among them J11 RE12A, J12 RS485_airdata, Q3 NPN, U8 MAX3485, U9 MOUDLE-SEEEDUINO-XIAO-ESP32C3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

Commit message: 2026/01
2026/01
Parts:
- removed DPS311: Adafruit DPS310, Connector_PinHeader_2.54mm:PinHeader_1x07_P2.54mm_Vertical, symbol New_Library:Adafruit_DPS310
- removed R28: 10k, Resistor_SMD:R_0603_1608Metric_Pad0.98x0.95mm_HandSolder, symbol Device:R
- R25: value 10k -> 20k
Connections:
- net encoder_raw: now also Q3.1 (B), R29.2
- no-connect marks 14 -> 13
Other:
- note added: "1. airdata"

Commit message: 0206
Parts:
- added R14, R6: 2k, Resistor_SMD:R_0603_1608Metric_Pad0.98x0.95mm_HandSolder, symbol Device:R
Connections:
- net +3.3V: now also R14.1, R6.1
- net SCL: now also R6.2
- net SDA: now also R14.2

Commit message: 0206_2
Connections:
- net SCL: now also AS5603.4 (SCL); no longer AS5602.4 (SCL)
- net SCL_soft: now also AS5602.4 (SCL); no longer AS5603.4 (SCL)
- net SDA: now also AS5603.5 (SDA); no longer AS5602.5 (SDA)
- net SDA_soft: now also AS5602.5 (SDA); no longer AS5603.5 (SDA)
Other:
- moved on the sheet: R14, R6
Changed lines of the file:
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@@
 	)
 	(junction
-		(at 69.85 62.23)
+		(at 101.6 162.56)
 		(diameter 0)
 		(color 0 0 0 0)
 	)
 	(junction
-		(at 107.95 139.7)
+		(at 69.85 62.23)
 		(diameter 0)
 		(color 0 0 0 0)
@@
 		(color 0 0 0 0)
 	)
-	(junction
-		(at 100.33 142.24)
-		(diameter 0)
-		(color 0 0 0 0)
-	)
 	(no_connect
 		(at 110.49 149.86)
@@
 	(wire
 		(pts
-			(xy 100.33 142.24) (xy 110.49 142.24)
+			(xy 53.34 113.03) (xy 66.04 113.03)
 		)
 		(stroke
@@
 	(wire
 		(pts
-			(xy 107.95 139.7) (xy 110.49 139.7)
+			(xy 105.41 139.7) (xy 110.49 139.7)
 		)
 		(stroke
@@
 	(wire
 		(pts
-			(xy 53.34 113.03) (xy 66.04 113.03)
+			(xy 138.43 119.38) (xy 138.43 129.54)
 		)
 		(stroke
@@
 	(wire
 		(pts
-			(xy 105.41 139.7) (xy 107.95 139.7)
+			(xy 54.61 68.58) (xy 62.23 68.58)
 		)
 		(stroke
@@
 	(wire
 		(pts
-			(xy 138.43 119.38) (xy 138.43 129.54)
+			(xy 130.81 99.06) (xy 130.81 97.79)
 		)
 		(stroke
@@
 	(wire
 		(pts
-			(xy 54.61 68.58) (xy 62.23 68.58)
+			(xy 133.35 119.38) (xy 133.35 121.92)
 		)
 		(stroke
@@
 	(wire
 		(pts
-			(xy 130.81 99.06) (xy 130.81 97.79)
+			(xy 55.88 109.22) (xy 55.88 115.57)
 		)
 		(stroke
@@
 	(wire
 		(pts
-			(xy 133.35 119.38) (xy 133.35 121.92)
+			(xy 93.98 161.29) (xy 93.98 165.1)
 		)
 		(stroke
@@
 	(wire
 		(pts
-			(xy 55.88 109.22) (xy 55.88 115.57)
+			(xy 69.85 60.96) (xy 69.85 62.23)
 		)
 		(stroke
@@
 	(wire
 		(pts
-			(xy 100.33 134.62) (xy 100.33 142.24)
+			(xy 128.27 121.92) (xy 129.54 121.92)
 		)
 		(stroke
@@
 	(wire
 		(pts
-			(xy 69.85 60.96) (xy 69.85 62.23)
+			(xy 43.18 120.65) (xy 66.04 120.65)
 		)
 		(stroke
@@
 	(wire
 		(pts
-			(xy 128.27 121.92) (xy 129.54 121.92)
+			(xy 69.85 62.23) (xy 69.85 63.5)
 		)
 		(stroke
@@
 	(wire
 		(pts
-			(xy 43.18 120.65) (xy 66.04 120.65)
+			(xy 110.49 76.2) (xy 110.49 99.06)
 		)
 		(stroke
@@
 	(wire
 		(pts
-			(xy 69.85 62.23) (xy 69.85 63.5)
+			(xy 93.98 165.1) (xy 110.49 165.1)
 		)
 		(stroke
@@
 	(wire
 		(pts
-			(xy 110.49 76.2) (xy 110.49 99.06)
+			(xy 99.06 170.18) (xy 110.49 170.18)
 		)
 		(stroke
@@
 	(wire
 		(pts
-			(xy 99.06 170.18) (xy 110.49 170.18)
+			(xy 100.33 162.56) (xy 101.6 162.56)
 		)
 		(stroke
@@
 	(wire
 		(pts
-			(xy 107.95 134.62) (xy 107.95 139.7)
+			(xy 101.6 161.29) (xy 101.6 162.56)
 		)
 		(stroke
@@
 	(wire
 		(pts
+			(xy 101.6 162.56) (xy 110.49 162.56)
+		)
+		(stroke
+			(width 0)
+			(type default)
+		)
+	)
+	(wire
+		(pts
 			(xy 135.89 99.06) (xy 152.4 99.06)
 		)
@@
 	(wire
 		(pts
-			(xy 99.06 142.24) (xy 100.33 142.24)
+			(xy 99.06 142.24) (xy 110.49 142.24)
 		)
 		(stroke
@@
 	(hierarchical_label "SDA_soft"
 		(shape input)
-		(at 110.49 162.56 180)
+		(at 105.41 139.7 180)
 		(effects
 			(font
@@
 	(hierarchical_label "SCL_soft"
 		(shape input)
-		(at 110.49 165.1 180)
+		(at 99.06 142.24 180)
 		(effects
 			(font
@@
 	(hierarchical_label "SCL"
 		(shape input)
-		(at 99.06 142.24 180)
+		(at 93.98 165.1 180)
 		(effects
 			(font
@@
 	(hierarchical_label "SDA"
 		(shape input)
-		(at 105.41 139.7 180)
+		(at 100.33 162.56 180)
 		(effects
 			(font
@@
 	(symbol
 		(lib_id "power:+3.3V")
-		(at 100.33 127 0)
+		(at 93.98 153.67 0)
 		(mirror y)
 		(unit 1)
@@
 		(on_board yes)
 		(dnp no)
-		(fields_autoplaced yes)
 		(property "Reference" "#PWR032"
-			(at 100.33 130.81 0)
+			(at 93.98 157.48 0)
 			(effects
 				(font
@@
 		)
 		(property "Value" "+3.3V"
-			(at 100.3299 123.19 90)
+			(at 93.9799 149.86 0)
 			(effects
 				(font
@@
 		)
 		(property "Footprint" ""
-			(at 100.33 127 0)
+			(at 93.98 153.67 0)
 			(effects
 				(font
@@
 		)
 		(property "Datasheet" ""
-			(at 100.33 127 0)
+			(at 93.98 153.67 0)
 			(effects
 				(font
@@
 		)
 		(property "Description" "Power symbol creates a global label with name \"+3.3V\""
-			(at 100.33 127 0)
+			(at 93.98 153.67 0)
 			(effects
 				(font
@@
 		)
 		(property "Value" "GND"
-			(at 94.488 167.64 0)
+			(at 94.488 167.64 90)
 			(effects
 				(font
@@
 	(symbol
 		(lib_id "Device:R")
-		(at 100.33 130.81 0)
+		(at 93.98 157.48 0)
 		(unit 1)
 		(exclude_from_sim no)
@@
 		(dnp no)
 		(property "Reference" "R6"
-			(at 102.87 130.81 90)
+			(at 96.52 157.48 90)
 			(effects
 				(font
@@
 		)
 		(property "Value" "2k"
-			(at 101.6 127.762 90)
+			(at 95.25 154.432 90)
 			(effects
 				(font
@@
 		)
 		(property "Footprint" "Resistor_SMD:R_0603_1608Metric_Pad0.98x0.95mm_HandSolder"
-			(at 98.552 130.81 90)
+			(at 92.202 157.48 90)
 			(effects
 				(font
@@
 		)
 		(property "Datasheet" "~"
-			(at 100.33 130.81 0)
+			(at 93.98 157.48 0)
 			(effects
 				(font
@@
 		)
 		(property "Description" "Resistor"
-			(at 100.33 130.81 0)
+			(at 93.98 157.48 0)
 			(effects
 				(font
@@
 	(symbol
 		(lib_id "Device:R")
-		(at 107.95 130.81 0)
+		(at 101.6 157.48 0)
 		(unit 1)
 		(exclude_from_sim no)
@@
 		(dnp no)
 		(property "Reference" "R14"
-			(at 110.49 130.81 90)
+			(at 104.14 157.48 90)
 			(effects
 				(font
@@
 		)
 		(property "Value" "2k"
-			(at 109.22 127.762 90)
+			(at 102.87 154.432 90)
 			(effects
 				(font
@@
 		)
 		(property "Footprint" "Resistor_SMD:R_0603_1608Metric_Pad0.98x0.95mm_HandSolder"
-			(at 106.172 130.81 90)
+			(at 99.822 157.48 90)
 			(effects
 				(font
@@
 		)
 		(property "Datasheet" "~"
-			(at 107.95 130.81 0)
+			(at 101.6 157.48 0)
 			(effects
 				(font
@@
 		)
 		(property "Description" "Resistor"
-			(at 107.95 130.81 0)
+			(at 101.6 157.48 0)
 			(effects
 				(font
@@
 	(symbol
 		(lib_id "power:+3.3V")
-		(at 107.95 127 0)
+		(at 101.6 153.67 0)
 		(mirror y)
 		(unit 1)
@@
 		(on_board yes)
 		(dnp no)
-		(fields_autoplaced yes)
 		(property "Reference" "#PWR033"
-			(at 107.95 130.81 0)
+			(at 101.6 157.48 0)
 			(effects
 				(font
@@
 		)
 		(property "Value" "+3.3V"
-			(at 107.9499 123.19 90)
+			(at 101.5999 149.86 0)
 			(effects
 				(font
@@
 		)
 		(property "Footprint" ""
-			(at 107.95 127 0)
+			(at 101.6 153.67 0)
 			(effects
 				(font
@@
 		)
 		(property "Datasheet" ""
-			(at 107.95 127 0)
+			(at 101.6 153.67 0)
 			(effects
 				(font
@@
 		)
 		(property "Description" "Power symbol creates a global label with name \"+3.3V\""
-			(at 107.95 127 0)
+			(at 101.6 153.67 0)
 			(effects
 				(font
