File: Kicad/boards/untitled.kicad_sch (KiCad schematic)
At the start: 18 parts, among them J11 RE12A, J12 RS485_airdata, Q3 NPN, U8 MAX3485, U9 MOUDLE-SEEEDUINO-XIAO-ESP32C3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

Commit message: edited boards
Parts:
- added R35, R36: 220k, Resistor_SMD:R_0603_1608Metric_Pad0.98x0.95mm_HandSolder, symbol Device:R
Connections:
- net +3.3V-1: now also R26.1, R27.1
- net +BATT-1: now also R35.1
- net GND-1: now also R36.2
- net V_check-1: now reaches U9.2 (GPIO3_A1_D1)
- net V_check-1: now also R35.2, R36.1
- removed net +5V: R26.1, R27.1, U9.14 (5V)

Commit message: edited boards
Connections:
- net encoder_out: now also U9.9 (GPIO8_D8_SCK); no longer U9.10 (GPIO9_D9_MISO)
Changed lines of the file:
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@@
 	)
 	(no_connect
-		(at 152.4 72.39)
+		(at 152.4 68.58)
 	)
 	(no_connect
@@
 	(hierarchical_label "encoder_out"
 		(shape input)
-		(at 152.4 68.58 0)
+		(at 152.4 72.39 0)
 		(effects
 			(font
@@
 		)
 		(property "Value" "330"
-			(at 46.482 114.3 90)
+			(at 54.102 113.284 90)
 			(effects
 				(font
@@
 		)
 		(property "Value" "3k"
-			(at 46.482 116.84 90)
+			(at 53.34 115.824 90)
 			(effects
 				(font
@@
 		)
 		(property "Value" "20k"
-			(at 52.578 110.49 90)
-			(effects
-				(font
+			(at 54.102 109.22 90)
+			(effects
+				(font
