File: Kicad/boards/_autosave-loggerboard.kicad_sch (KiCad schematic)
At the start: 21 parts, among them J2 Micro_SD_Card, J7 RS485_logger_2, J8 RS485_logger, J9 BNO085, U2 MAX3485, U5 MOUDLE-SEEEDUINO-XIAO-ESP32C3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, U6 DS3231MZ

Commit message: 電源1つに
Parts:
- R4: value 2k -> 680
Connections:
- net +3.3V is gone; now on net +3.3V-2: J9.JP1_1 (VIN)
- net +BATT renamed +BATT-2
- net GND renamed GND-2
