File: Kicad/boards/_autosave-untitled.kicad_sch (KiCad schematic)
At the start: 18 parts, among them J11 RE12A, J12 RS485_airdata, Q3 NPN, U8 MAX3485, U9 MOUDLE-SEEEDUINO-XIAO-ESP32C3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

Commit message: 電源1つに
Connections:
- net +BATT renamed +BATT-1
- net GND renamed GND-1
