File: Kicad/boards/26proto.kicad_pcb (KiCad board)
At the start: 2 copper layers, 98.8 x 93.1 mm, 67 parts, among them J1 5051104096, J10 Conn_01x05, J2 Micro_SD_Card, J3 URM37, J4 RE12A, J5 RS485_TFT, J6 RS485_airdata, J7 RS485_logger_2, J8 RS485_logger, J9 BNO085, Q2 NPN, SW1 SW_DIP_x01, U1 MOUDLE-SEEEDUINO-XIAO-ESP32C3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, U11 MOUDLE-SEEEDUINO-XIAO-ESP32C3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, U2 MAX3485, U3 1339D, U4 MAX3485, U5 MOUDLE-SEEEDUINO-XIAO-ESP32C3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, U6 MAX3485, U7 MOUDLE-SEEEDUINO-XIAO-ESP32C3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, Y1 CFS-206

Commit message: 一旦完成
Other:
- board text added: "AoAセンサ"
- board text added: "AoSセンサ"
- board text added: "DPS310"
- board text added: "RE12A"
- board text added: "RS485"
- board text added: "URM37"
- board text added: "舵角計"

Commit message: edited
Parts:
- added AS5602: AoS, Connector_PinHeader_2.54mm:PinHeader_1x06_P2.54mm_Vertical, F.Cu at (103.6, 56.8)
- added AS5603: AoA, Connector_PinHeader_2.54mm:PinHeader_1x06_P2.54mm_Vertical, F.Cu at (108.2, 56.8)
- added Batt4: Conn_01x02, Connector_JST:JST_PH_S2B-PH-SM4-TB_1x02-1MP_P2.00mm_Horizontal, F.Cu at (115.7, 60.1)
- added D4: LED, LED_SMD:LED_0603_1608Metric_Pad1.05x0.95mm_HandSolder, F.Cu at (97.3, 59.9)
- added DPS311: Adafruit DPS310, Connector_PinHeader_2.54mm:PinHeader_1x07_P2.54mm_Vertical, F.Cu at (83.6, 54.3)
- added J11: RE12A, Connector_JST:JST_XH_S4B-XH-SM4-TB_1x04-1MP_P2.50mm_Horizontal, F.Cu at (110.2, 34.9)
- added J12: RS485_airdata, Connector_JST:JST_XH_S4B-XH-SM4-TB_1x04-1MP_P2.50mm_Horizontal, F.Cu at (110.2, 48.0)
- added Q3: NPN, Package_TO_SOT_SMD:SOT-23, F.Cu at (92.7, 61.0)
- added R25: 10k, Resistor_SMD:R_0603_1608Metric_Pad0.98x0.95mm_HandSolder, F.Cu at (88.0, 53.3)
- added R26: 330, Resistor_SMD:R_0603_1608Metric_Pad0.98x0.95mm_HandSolder, F.Cu at (88.0, 55.8)
- added R27: 3k, Resistor_SMD:R_0603_1608Metric_Pad0.98x0.95mm_HandSolder, F.Cu at (88.0, 58.3)
- added R28: 10k, Resistor_SMD:R_0603_1608Metric_Pad0.98x0.95mm_HandSolder, F.Cu at (88.0, 60.8)
- added R29: 100k, Resistor_SMD:R_0603_1608Metric_Pad0.98x0.95mm_HandSolder, F.Cu at (88.0, 63.3)
- added R30: 10k, Resistor_SMD:R_0603_1608Metric_Pad0.98x0.95mm_HandSolder, F.Cu at (88.0, 65.8)
- added R31: 100, Resistor_SMD:R_0603_1608Metric_Pad0.98x0.95mm_HandSolder, F.Cu at (88.0, 68.3)
- added R32: 120, Resistor_SMD:R_0603_1608Metric_Pad0.98x0.95mm_HandSolder, F.Cu at (88.0, 70.9)
- added U8: MAX3485, Package_SO:SOIC-8_3.9x4.9mm_P1.27mm, F.Cu at (94.4, 55.4)
- added U9: MOUDLE-SEEEDUINO-XIAO-ESP32C3_airdata, footprints:XIAO-ESP32C3-SMD, F.Cu at (91.3, 40.9)
Connections:
- BT1 pad 2: encoder_cathode -> GND
- Batt1 pad 2: encoder_cathode -> GND
- Batt2 pad 2: encoder_cathode -> GND
- C1 pad 2: encoder_cathode -> GND
- D1 pad 1: encoder_cathode -> GND
- D2 pad 1: encoder_cathode -> GND
- J1 pad 1: encoder_cathode -> GND
- J1 pad 31: encoder_cathode -> GND
- J1 pad 34: encoder_cathode -> GND
- J1 pad 35: encoder_cathode -> GND
- J1 pad 36: encoder_cathode -> GND
- J1 pad 37: encoder_cathode -> GND
- J1 pad 39: encoder_cathode -> GND
- J10 pad 2: encoder_cathode -> GND
- J2 pad 6: encoder_cathode -> GND
- J2 pad 9: encoder_cathode -> GND
- J3 pad 2: encoder_cathode -> GND
- J5 pad 2: encoder_cathode -> GND
- J7 pad 2: encoder_cathode -> GND
- J8 pad 2: encoder_cathode -> GND
- J9 pad JP1_3: encoder_cathode -> GND
- R18 pad 2: encoder_cathode -> GND
- R19 pad 2: encoder_cathode -> GND
- R9 pad 2: encoder_cathode -> GND
- U1 pad 13: encoder_cathode -> GND
- U1 pad 16: encoder_cathode -> GND
- U11 pad 13: encoder_cathode -> GND
- U11 pad 16: encoder_cathode -> GND
- U2 pad 5: encoder_cathode -> GND
- U3 pad 4: encoder_cathode -> GND
- U4 pad 5: encoder_cathode -> GND
- U5 pad 13: encoder_cathode -> GND
- U5 pad 16: encoder_cathode -> GND
Routing:
- net GND: track 0.00 -> 59.3 mm, vias 0 -> 2
- net encoder_cathode: track 319.8 -> 260.5 mm, vias 9 -> 7

Commit message: 0206
Parts:
- removed Q2: NPN, Package_TO_SOT_SMD:SOT-23
- removed R15: 100k, Resistor_SMD:R_0603_1608Metric_Pad0.98x0.95mm_HandSolder
- removed R16: 10k, Resistor_SMD:R_0603_1608Metric_Pad0.98x0.95mm_HandSolder
- removed U7: MOUDLE-SEEEDUINO-XIAO-ESP32C3_airdata, footprints:XIAO-ESP32C3-SMD
- added BT2: MS621, Battery:BatteryHolder_Seiko_MS621F, F.Cu at (-16.5, 106.7)
- added Batt2: Conn_01x02, Connector_JST:JST_PH_S2B-PH-SM4-TB_1x02-1MP_P2.00mm_Horizontal, F.Cu at (-19.6, 82.0)
- added C1: 0.1uF, Capacitor_SMD:C_0603_1608Metric_Pad1.08x0.95mm_HandSolder, F.Cu at (-47.1, 108.5)
- added C2: 47uF, Capacitor_SMD:C_0603_1608Metric_Pad1.08x0.95mm_HandSolder, F.Cu at (-47.1, 111.0)
- added D1: LED, LED_SMD:LED_0603_1608Metric_Pad1.05x0.95mm_HandSolder, F.Cu at (-27.0, 40.9)
- added D2: LED, LED_SMD:LED_0603_1608Metric_Pad1.05x0.95mm_HandSolder, F.Cu at (-47.1, 106.0)
- added D5: D, Diode_SMD:Nexperia_CFP3_SOD-123W, F.Cu at (-46.5, 103.1)
- added DPS311: Adafruit DPS310, Connector_PinHeader_2.54mm:PinHeader_1x07_P2.54mm_Vertical, F.Cu at (-25.1, 54.4)
- added J10: Conn_01x04, Connector_JST:JST_PH_S4B-PH-SM4-TB_1x04-1MP_P2.00mm_Horizontal, F.Cu at (-34.6, 57.7)
- added J2: Micro_SD_Card, Connector_Card:microSD_HC_Hirose_DM3AT-SF-PEJM5, F.Cu at (-34.1, 111.8)
- added J3: URM37, Connector_JST:JST_XH_S4B-XH-SM4-TB_1x04-1MP_P2.50mm_Horizontal, F.Cu at (-60.5, 50.1)
- added J5: RS485_TFT, Connector_JST:JST_XH_S4B-XH-SM4-TB_1x04-1MP_P2.50mm_Horizontal, F.Cu at (-60.5, 63.1)
- added J7: RS485_logger_2, Connector_JST:JST_XH_S4B-XH-SM4-TB_1x04-1MP_P2.50mm_Horizontal, F.Cu at (-33.6, 82.9)
- added J8: RS485_logger, Connector_JST:JST_XH_S4B-XH-SM4-TB_1x04-1MP_P2.50mm_Horizontal, F.Cu at (-33.6, 95.9)
- added JP1: SolderJumper_2_Open, Jumper:SolderJumper-2_P1.3mm_Open_TrianglePad1.0x1.5mm, F.Cu at (-55.8, 71.4)
- added R1: 10k, Resistor_SMD:R_0603_1608Metric_Pad0.98x0.95mm_HandSolder, F.Cu at (-47.1, 113.5)
- added R10: 3.3k, Resistor_SMD:R_0603_1608Metric_Pad0.98x0.95mm_HandSolder, F.Cu at (-20.7, 58.3)
- added R11: 3.3k, Resistor_SMD:R_0603_1608Metric_Pad0.98x0.95mm_HandSolder, F.Cu at (-20.7, 60.8)
- added R12: 3.3k, Resistor_SMD:R_0603_1608Metric_Pad0.98x0.95mm_HandSolder, F.Cu at (-20.7, 63.4)
- added R13: 10k, Resistor_SMD:R_0603_1608Metric_Pad0.98x0.95mm_HandSolder, F.Cu at (-47.1, 121.1)
- added R17: 2, Resistor_THT:R_Axial_DIN0207_L6.3mm_D2.5mm_P7.62mm_Horizontal, F.Cu at (-40.1, 72.3)
- added R18: 10k, Resistor_SMD:R_0603_1608Metric_Pad0.98x0.95mm_HandSolder, F.Cu at (-20.7, 65.9)
- added R2: 10k, Resistor_SMD:R_0603_1608Metric_Pad0.98x0.95mm_HandSolder, F.Cu at (-47.1, 116.1)
- added R20: 3.3k, Resistor_SMD:R_0603_1608Metric_Pad0.98x0.95mm_HandSolder, F.Cu at (-20.7, 68.4)
- added R22: 100, Resistor_SMD:R_0603_1608Metric_Pad0.98x0.95mm_HandSolder, F.Cu at (-47.1, 123.6)
- added R23: 100, Resistor_SMD:R_0603_1608Metric_Pad0.98x0.95mm_HandSolder, F.Cu at (-20.7, 70.9)
- added R3: 10k, Resistor_SMD:R_0603_1608Metric_Pad0.98x0.95mm_HandSolder, F.Cu at (-47.1, 118.6)
- added R4: 2k, Resistor_THT:R_Axial_DIN0207_L6.3mm_D2.5mm_P7.62mm_Horizontal, F.Cu at (-24.1, 112.9)
- added R5: 120, Resistor_SMD:R_0603_1608Metric_Pad0.98x0.95mm_HandSolder, F.Cu at (-20.7, 53.3)
- added R6: 2k, Resistor_SMD:R_0603_1608Metric_Pad0.98x0.95mm_HandSolder, F.Cu at (-12.5, 21.9)
- added R7: 2k, Resistor_THT:R_Axial_DIN0207_L6.3mm_D2.5mm_P7.62mm_Horizontal, F.Cu at (-24.1, 117.0)
- added R8: 2k, Resistor_THT:R_Axial_DIN0207_L6.3mm_D2.5mm_P7.62mm_Horizontal, F.Cu at (-24.1, 121.0)
- added R9: 10k, Resistor_SMD:R_0603_1608Metric_Pad0.98x0.95mm_HandSolder, F.Cu at (-20.7, 55.8)
- added SW1: SW_DIP_x01, footprints:CLSB12A02T, F.Cu at (-36.4, 66.6)
- added U2: MAX3485, Package_SO:SOIC-8_3.9x4.9mm_P1.27mm, F.Cu at (-20.5, 91.0)
- added U3: 1339D, Package_SO:TSSOP-8_3x3mm_P0.65mm, F.Cu at (-65.9, 72.0)
- added U4: MAX3485, Package_SO:SOIC-8_3.9x4.9mm_P1.27mm, F.Cu at (-20.3, 46.9)
- added Y1: CFS-206, Crystal:Crystal_DS26_D2.0mm_L6.0mm_Vertical, F.Cu at (-61.2, 71.7)
- Batt1: moved to F.Cu
- Batt4, R29: moved to B.Cu
- J4: value RE12A -> Conn_01x03 servo; footprint Connector_JST:JST_XH_S4B-XH-SM4-TB_1x04-1MP_P2.50mm_Horizontal -> Connector_JST:JST_PH_S3B-PH-K_1x03_P2.00mm_Horizontal
- J6: value RS485_airdata -> Conn_01x03 encoder_direct; footprint Connector_JST:JST_XH_S4B-XH-SM4-TB_1x04-1MP_P2.50mm_Horizontal -> Connector_JST:JST_PH_S3B-PH-K_1x03_P2.00mm_Horizontal
- R14: value 10k -> 2k
- R25: value 10k -> 20k
- U6: value MAX3485 -> DS3231MZ
- moved J4 283.9 mm to (-48.7, 54.4)
- moved J6 276.8 mm to (-48.7, 64.1), turned to 0 degrees
- moved Batt1 276.7 mm to (-24.1, 25.5)
- moved R14 253.8 mm to (-12.5, 26.0), turned to 0 degrees
- moved U6 253.7 mm to (-20.5, 97.5), turned to 0 degrees
- moved R28 147.4 mm to (228.5, 105.4), turned to 90 degrees
- moved U9 147.1 mm to (229.1, 92.4), turned to -90 degrees
- moved R29 143.1 mm to (225.0, 104.9), turned to -90 degrees
- moved J11 142.5 mm to (228.9, 113.8)
- moved Q3 136.1 mm to (221.5, 104.9), turned to 90 degrees
- moved R30 134.7 mm to (216.1, 107.5)
- moved U8 133.9 mm to (228.0, 46.4), turned to 180 degrees
- moved Batt4 133.8 mm to (238.0, 114.4)
- moved R31 130.6 mm to (211.1, 112.0)
- moved R32 130.6 mm to (211.1, 114.5)
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Connections:
- net CS renamed /3. TFT/CS
- net DCX-SCLK renamed /3. TFT/DCX-SCLK
- net Net-(U8-DE) renamed /1. airdata/DE/RE
- net RES renamed /3. TFT/RES
- net SDA-MOSI renamed /3. TFT/SDA-MOSI
- net SDO-MISO renamed /3. TFT/SDO-MISO
- net WRX-D/C renamed /3. TFT/WRX-D/C
- AS5602 pad 2: pot_Vin -> +3.3V
- AS5603 pad 2: pot_Vin -> +3.3V
- J1 pad 32: pot_Vin -> +3.3V
- J1 pad 33: pot_Vin -> +3.3V
- J1 pad 7: pot_Vin -> +3.3V
- J1 pad 8: pot_Vin -> +3.3V
- J4 pad 1: Net-(J4-Pin_1) -> +3.3V
- J4 pad 2: Net-(J4-Pin_2) -> GND
- J4 pad 3: encoder_cathode -> /3. TFT/servo
- J6 pad 1: unconnected-(J6-Pin_1-Pad1) -> +3.3V
- J6 pad 2: encoder_cathode -> GND
- J6 pad 3: RS485_A -> /3. TFT/RX_encoder
- J9 pad JP1_1: pot_Vin -> +3.3V
- J9 pad JP1_4: SCL_BNO085 -> /2.logger/SCL
- J9 pad JP1_5: SDA_BNO085 -> /2.logger/SDA
- Q3 pad 1: Net-(Q3-B) -> /1. airdata/encoder_raw
- R14 pad 1: encoder_raw -> +3.3V
- R14 pad 2: Net-(Q2-B) -> /1. airdata/SDA
- R29 pad 2: Net-(Q3-B) -> /1. airdata/encoder_raw
- R30 pad 1: pot_Vin -> +3.3V
- U1 pad 12: pot_Vin -> +3.3V
- U1 pad 4: Net-(U1-GPIO5_A3_D3) -> /3. TFT/DE/RE
- U1 pad 5: SDA_board3 -> /3. TFT/SDA
- U1 pad 6: SCL_board3 -> /3. TFT/SCL
- U11 pad 1: Pot_elv -> /3. TFT/Pot_elv
- U11 pad 10: unconnected-(U11-GPIO9_D9_MISO-Pad10) -> /3. TFT/servo
- U11 pad 12: pot_Vin -> +3.3V
- U11 pad 2: Pot_rud -> /3. TFT/Pot_rud
- U11 pad 3: Pot_trim -> /3. TFT/Pot_trim
- U11 pad 5: SDA_board3 -> /3. TFT/SDA
- U11 pad 6: SCL_board3 -> /3. TFT/SCL
- U11 pad 7: TX_URM37 -> /3. TFT/TX
- U11 pad 8: RX_URM37 -> /3. TFT/RX
- U11 pad 9: unconnected-(U11-GPIO8_D8_SCK-Pad9) -> /3. TFT/RX_encoder
- U5 pad 1: Net-(U2-DE) -> unconnected-(U5-GPIO2_A0_D0-Pad1)
- U5 pad 10: MISO_SD -> /2.logger/MISO
- U5 pad 11: MOSI_SD -> /2.logger/MOSI
- U5 pad 12: pot_Vin -> +3.3V
- U5 pad 3: unconnected-(U5-GPIO4_A2_D2-Pad3) -> /2.logger/DE/RE
- U5 pad 4: CS_SD -> /2.logger/CS
- U5 pad 5: SDA_BNO085 -> /2.logger/SDA
- U5 pad 6: SCL_BNO085 -> /2.logger/SCL
- U5 pad 9: SCLK_SD -> /2.logger/SCLK
- U6 pad 1: Net-(U6-RO) -> unconnected-(U6-32KHZ-Pad1)
- U6 pad 2: Net-(U6-DE) -> +3.3V
- U6 pad 3: Net-(U6-DE) -> unconnected-(U6-~{INT}/SQW-Pad3)
- U6 pad 4: Net-(U6-DI) -> unconnected-(U6-~{RST}-Pad4)
- U6 pad 5: encoder_cathode -> GND
- U6 pad 6: RS485_A -> Net-(BT2--)
- U6 pad 7: RS485_B -> /2.logger/SDA
- U6 pad 8: pot_Vin -> /2.logger/SCL
- U8 pad 8: pot_Vin -> +3.3V
- U9 pad 12: pot_Vin -> +3.3V
Routing:
- net +3.3V: track 0.00 -> 128.3 mm
- net pot_Vin: track 344.3 -> 216.0 mm
- net Net-(U8-RO): track 0.00 -> 81.3 mm, vias 0 -> 2
- net Net-(U6-RO): track 81.3 -> 0.00 mm, vias 2 -> 0
- net Net-(U6-DE): track 79.4 -> 0.00 mm, vias 2 -> 0
- net /1. airdata/DE/RE: track 0.00 -> 79.4 mm, vias 0 -> 2
- net Net-(U8-DI): track 0.00 -> 55.8 mm, vias 0 -> 2
- net Net-(U6-DI): track 55.8 -> 0.00 mm, vias 2 -> 0
- net encoder_cathode: track 260.5 -> 230.9 mm, vias 7 -> 5
- net GND: track 59.3 -> 88.9 mm, vias 2 -> 4
- net SCL_BNO085: track 27.2 -> 0.00 mm
- net /2.logger/SCL: track 0.00 -> 27.2 mm
- net SDA_BNO085: track 25.8 -> 0.00 mm, vias 1 -> 0
- net /2.logger/SDA: track 0.00 -> 25.8 mm, vias 0 -> 1
- net Net-(Q3-B): track 0.00 -> 11.3 mm
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
Commit message: 0206_2
Parts:
- removed AS5600: AoS, Connector_PinHeader_2.54mm:PinHeader_1x06_P2.54mm_Vertical
- removed AS5601: AoA, Connector_PinHeader_2.54mm:PinHeader_1x06_P2.54mm_Vertical
- removed the Batt2 at (194.7, 112.4)
- removed Batt3: Conn_01x02, Connector_JST:JST_PH_S2B-PH-SM4-TB_1x02-1MP_P2.00mm_Horizontal
- removed the D2 at (191.0, 88.0)
- removed DPS310: Adafruit DPS310, Connector_PinHeader_2.54mm:PinHeader_1x07_P2.54mm_Vertical
- removed the DPS311 at (188.5, 51.9)
- removed the DPS311 at (-25.1, 54.4)
- removed the J10 at (179.1, 76.8)
- removed the J2 at (192.4, 97.8)
- removed the J3 at (196.1, 76.0)
- removed the J5 at (162.1, 76.0)
- removed the J7 at (192.6, 103.4)
- removed the J8 at (152.9, 103.7)
- removed the JP1 at (-55.8, 71.4)
- removed the R10 at (179.0, 67.0)
- removed the R17 at (162.8, 32.5)
- removed the R18 at (181.0, 60.0)
- removed R19, R28: 10k, Resistor_SMD:R_0603_1608Metric_Pad0.98x0.95mm_HandSolder
- removed R21: 3.3k, Resistor_SMD:R_0603_1608Metric_Pad0.98x0.95mm_HandSolder
- removed the R22 at (186.0, 88.0)
- removed the R4 at (223.0, 46.4)
- removed the R6 at (221.5, 104.9)
- removed the SW1 at (150.5, 39.0)
- removed the U2 at (-20.5, 91.0)
- removed U3 (x2): 1339D, Package_SO:TSSOP-8_3x3mm_P0.65mm
- removed the U4 at (171.7, 63.5)
- removed Y1 (x2): CFS-206, Crystal:Crystal_DS26_D2.0mm_L6.0mm_Vertical
- added DPS311: Adafruit DPS310, Connector_PinHeader_2.54mm:PinHeader_1x07_P2.54mm_Vertical, F.Cu at (189.0, 55.9)
- added J13: Conn_01x03 speaker, Connector_JST:JST_PH_S3B-PH-K_1x03_P2.00mm_Horizontal, B.Cu at (189.0, 24.4)
- AS5603, Batt1, Batt2, J2, R18, R6, R9: moved to B.Cu
- J10: footprint Connector_JST:JST_PH_S4B-PH-SM4-TB_1x04-1MP_P2.00mm_Horizontal -> Connector_JST:JST_XH_S4B-XH-SM4-TB_1x04-1MP_P2.50mm_Horizontal
- J4, J6: footprint Connector_JST:JST_PH_S3B-PH-K_1x03_P2.00mm_Horizontal -> Connector_JST:JST_PH_B3B-PH-K_1x03_P2.00mm_Vertical
- R29, R9: moved to F.Cu
- R4: footprint Resistor_THT:R_Axial_DIN0207_L6.3mm_D2.5mm_P7.62mm_Horizontal -> Resistor_SMD:R_0603_1608Metric_Pad0.98x0.95mm_HandSolder
- R7, R8: footprint Resistor_THT:R_Axial_DIN0207_L6.3mm_D2.5mm_P7.62mm_Horizontal -> Resistor_SMD:R_0603_1608Metric_Pad0.98x0.95mm_HandSolder; moved to B.Cu
- moved J3 257.9 mm to (196.1, 76.0)
- moved J4 256.3 mm to (207.5, 64.0), turned to 180 degrees
- moved J6 256.3 mm to (207.5, 57.5), turned to 180 degrees
- moved R6 239.1 mm to (223.5, 60.0), turned to -90 degrees
- moved R14 238.4 mm to (224.1, 55.5)
- moved R22 235.8 mm to (186.0, 88.0), turned to -90 degrees
- moved D2 231.2 mm to (183.7, 92.5), turned to -90 degrees
- moved Batt1 229.8 mm to (200.0, 76.5), turned to 180 degrees
- moved J7 227.1 mm to (192.6, 103.4), turned to 90 degrees
- moved J2 226.9 mm to (192.4, 97.8), turned to -90 degrees
- moved J5 223.0 mm to (162.1, 76.0)
- moved D5 218.5 mm to (171.6, 117.0)
- moved Batt2 216.4 mm to (194.7, 112.4), turned to -90 degrees
- moved J10 214.4 mm to (179.1, 76.0)
- moved R17 206.8 mm to (162.8, 32.5), turned to 180 degrees
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Connections:
- AS5602 pad 4: /1. airdata/SCL -> /1. airdata/SCL_soft
- AS5602 pad 5: /1. airdata/SDA -> /1. airdata/SDA_soft
- AS5603 pad 4: /1. airdata/SCL_soft -> /1. airdata/SCL
- AS5603 pad 5: /1. airdata/SDA_soft -> /1. airdata/SDA
- U11 pad 4: unconnected-(U11-GPIO5_A3_D3-Pad4) -> /3. TFT/Speaker
- U2 pad 2: Net-(U2-DE) -> /2.logger/DE/RE
- U2 pad 3: Net-(U2-DE) -> /2.logger/DE/RE
- U2 pad 8: pot_Vin -> +3.3V
Routing:
- net encoder_cathode: track 230.9 -> 0.00 mm, vias 5 -> 0
- net GND: track 88.9 -> 295.8 mm, vias 4 -> 9
- net pot_Vin: track 216.0 -> 74.1 mm, vias 6 -> 2
- net +3.3V: track 128.3 -> 240.7 mm, vias 0 -> 3
- net SCL_airdata: track 57.2 -> 0.00 mm, vias 1 -> 0
- net /2.logger/SCL: track 27.2 -> 82.2 mm, vias 0 -> 1
- net SDA_airdata: track 53.7 -> 0.00 mm
- net /2.logger/SDA: track 25.8 -> 71.8 mm, vias 1 -> 2
- net Pot_elv: track 40.0 -> 0.00 mm, vias 2 -> 0
- net /3. TFT/Pot_elv: track 0.00 -> 39.5 mm, vias 0 -> 2
- net Pot_rud: track 36.9 -> 0.00 mm, vias 2 -> 0
- net /3. TFT/Pot_rud: track 0.00 -> 36.6 mm, vias 0 -> 2
- net Pot_trim: track 33.1 -> 0.00 mm, vias 2 -> 0
- net RX_URM37: track 31.4 -> 0.00 mm
- net /3. TFT/RX: track 0.00 -> 31.4 mm
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Other:
- board size 98.8 x 93.1 mm -> 98.8 x 95.5 mm

Commit message: 電源1つに
Parts:
- removed BT1: MS621, Battery:BatteryHolder_Seiko_MS621F
- removed the C1 at (188.7, 93.1)
- removed the D1 at (207.5, 70.0)
- removed D3: LED, LED_SMD:LED_0603_1608Metric_Pad1.05x0.95mm_HandSolder
- removed the R1 at (177.7, 102.1)
- removed the R11 at (-20.7, 60.8)
- removed the R12 at (188.1, 46.0)
- removed the R13 at (180.7, 97.4)
- removed the R2 at (177.5, 104.4)
- removed the R20 at (-19.9, 66.5)
- removed the R23 at (-14.9, 69.5)
- removed R24: 100, Resistor_SMD:R_0603_1608Metric_Pad0.98x0.95mm_HandSolder
- removed the R3 at (176.8, 99.9)
- removed the R5 at (-12.4, 51.5)
- removed the R7 at (239.0, 105.9)
- removed the R8 at (235.5, 105.8)
- removed the R9 at (-16.9, 53.5)
- removed the REF** at (149.7, 77.0)
- added C3: 47uF, Capacitor_SMD:C_0603_1608Metric_Pad1.08x0.95mm_HandSolder, B.Cu at (163.0, 41.6)
- R1, R13, R2, R3: moved to B.Cu
- R11, R12: value 3.3k -> 2k
- R4: value 2k -> 680
- moved C1 237.3 mm to (188.7, 93.1), turned to 90 degrees
- moved D1 236.3 mm to (207.5, 70.0), turned to 90 degrees
- moved C2 231.1 mm to (187.5, 96.9), turned to 90 degrees
- moved R1 229.8 mm to (177.7, 102.0), turned to 180 degrees
- moved R3 227.3 mm to (176.8, 99.9)
- moved R13 226.8 mm to (180.7, 97.4), turned to 180 degrees
- moved R2 217.6 mm to (177.5, 104.4), turned to 180 degrees
- moved R12 201.2 mm to (188.1, 46.0), turned to -90 degrees
- moved R26 126.4 mm to (239.0, 107.4), turned to -90 degrees
- moved R27 122.6 mm to (235.5, 107.3), turned to -90 degrees
- moved J13 62.5 mm to (151.5, 74.5), turned to 180 degrees
- moved R6 22.1 mm to (225.0, 82.0), turned to 180 degrees
- moved DPS311 15.6 mm to (189.0, 71.5), turned to 180 degrees
- moved R14 10.6 mm to (225.5, 66.0), turned to -90 degrees
- moved D2 8.57 mm to (191.0, 88.0)
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Connections:
- AS5602 pad 2: +3.3V -> +3.3V-1
- AS5602 pad 3: GND -> GND-1
- AS5603 pad 2: +3.3V -> +3.3V-1
- AS5603 pad 3: GND -> GND-1
- Batt1 pad 1: +BATT -> +BATT-3
- Batt1 pad 2: GND -> GND-3
- Batt2 pad 1: +BATT -> +BATT-2
- Batt2 pad 2: GND -> GND-2
- Batt4 pad 1: +BATT -> +BATT-1
- Batt4 pad 2: GND -> GND-1
- C1 pad 1: +3.3V -> +3.3V-2
- C1 pad 2: GND -> GND-2
- C2 pad 1: +3.3V -> +3.3V-2
- C2 pad 2: GND -> GND-2
- D1 pad 1: GND -> GND-3
- D2 pad 1: GND -> GND-2
- D4 pad 1: GND -> GND-1
- D5 pad 2: +3.3V -> +3.3V-2
- DPS311 pad 2: +3.3V -> +3.3V-3
- DPS311 pad 3: GND -> GND-3
- DPS311 pad 5: GND -> GND-3
- DPS311 pad 7: +3.3V -> unconnected-(DPS311-CS-Pad7)
- J1 pad 1: GND -> GND-3
- J1 pad 31: GND -> GND-3
- J1 pad 32: +3.3V -> +3.3V-3
- J1 pad 33: +3.3V -> +3.3V-3
- J1 pad 34: GND -> GND-3
- J1 pad 35: GND -> GND-3
- J1 pad 36: GND -> GND-3
- J1 pad 37: GND -> GND-3
- J1 pad 39: GND -> GND-3
- J1 pad 7: +3.3V -> +3.3V-3
- J1 pad 8: +3.3V -> +3.3V-3
- J10 pad 1: +3.3V -> +3.3V-3
- J10 pad 2: GND -> GND-3
- J11 pad 3: GND -> GND-1
- J11 pad 4: GND -> GND-1
- J12 pad 2: GND -> GND-1
- J13 pad 1: +3.3V -> +3.3V-3
- J13 pad 2: GND -> GND-3
- J2 pad 4: +3.3V -> +3.3V-2
- J2 pad 6: GND -> GND-2
- J2 pad 9: GND -> GND-2
- J3 pad 1: +3.3V -> +3.3V-3
- J3 pad 2: GND -> GND-3
- J4 pad 1: +3.3V -> +3.3V-3
- J4 pad 2: GND -> GND-3
- J5 pad 2: GND -> GND-3
- J6 pad 1: +3.3V -> +3.3V-3
- J6 pad 2: GND -> GND-3
- J7 pad 2: GND -> GND-2
- J8 pad 2: GND -> GND-2
- J9 pad JP1_1: +3.3V -> +3.3V-2
- J9 pad JP1_3: GND -> GND-2
- Q3 pad 2: GND -> GND-1
- R1 pad 2: +3.3V -> +3.3V-2
- R11 pad 1: SDA_board3 -> /3. TFT/SDA
- R11 pad 2: pot_Vin -> +3.3V-3
- R12 pad 1: +3.3V -> +3.3V-3
- R13 pad 2: +3.3V -> +3.3V-2
- R14 pad 1: +3.3V -> +3.3V-1
- R17 pad 1: +3.3V -> +3.3V-3
- R18 pad 2: GND -> GND-3
- R2 pad 2: +3.3V -> +3.3V-2
- R29 pad 1: GND -> GND-1
- R3 pad 2: +3.3V -> +3.3V-2
- R30 pad 1: +3.3V -> +3.3V-1
- R5 pad 1: RS485_B -> /3. TFT/RS485_B
- R5 pad 2: RS485_A -> /3. TFT/RS485_A
- R6 pad 1: +3.3V -> +3.3V-1
- R7 pad 1: +3.3V -> +3.3V-2
- R8 pad 1: +3.3V -> +3.3V-2
- R9 pad 2: GND -> GND-3
- U1 pad 12: +3.3V -> +3.3V-3
- U1 pad 13: GND -> GND-3
- U1 pad 15: +BATT -> unconnected-(U1-BAT-Pad15)
- U1 pad 16: GND -> GND-3
- U11 pad 12: +3.3V -> +3.3V-3
- U11 pad 13: GND -> GND-3
- U11 pad 15: +BATT -> +BATT-3
- U11 pad 16: GND -> GND-3
- U2 pad 5: GND -> GND-2
- U2 pad 8: +3.3V -> +3.3V-2
- U4 pad 5: GND -> GND-3
- U4 pad 8: +3.3V -> +3.3V-3
- U5 pad 12: +3.3V -> +3.3V-2
- U5 pad 13: GND -> GND-2
- U5 pad 15: +BATT -> +BATT-2
- U5 pad 16: GND -> GND-2
- U6 pad 2: +3.3V -> +3.3V-2
- U6 pad 5: GND -> GND-2
- U8 pad 5: GND -> GND-1
- U8 pad 8: +3.3V -> +3.3V-1
- U9 pad 12: +3.3V -> +3.3V-1
- U9 pad 13: GND -> GND-1
- U9 pad 15: +BATT -> +BATT-1
- U9 pad 16: GND -> GND-1
Routing:
- net GND: track 295.8 -> 0.00 mm, vias 9 -> 0
- net +3.3V: track 240.7 -> 0.00 mm, vias 3 -> 0
- net +3.3V-3: track 0.00 -> 205.1 mm
- net +BATT: track 191.3 -> 0.00 mm, vias 9 -> 0
- net GND-1: track 0.00 -> 177.1 mm, vias 0 -> 5
- net +3.3V-2: track 0.00 -> 92.9 mm, vias 0 -> 2
- net +BATT-2: track 0.00 -> 77.4 mm, vias 0 -> 4
- net +3.3V-1: track 0.00 -> 74.9 mm, vias 0 -> 3
- net pot_Vin: track 74.1 -> 0.00 mm, vias 2 -> 0
- net /3. TFT/Speaker: track 0.00 -> 69.2 mm, vias 0 -> 1
- net GND-2: track 0.00 -> 66.8 mm, vias 0 -> 4
- net GND-3: track 0.00 -> 54.9 mm, vias 0 -> 91
- net /1. airdata/SCL_soft: track 0.00 -> 52.3 mm, vias 0 -> 3
- net /3. TFT/SCL: track 0.00 -> 46.0 mm, vias 0 -> 2
- net CS_SD: track 44.7 -> 0.00 mm, vias 2 -> 0
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- added copper zone on B.Cu, net GND-1
- added copper zone on F.Cu, net GND-1
- added copper zone on B.Cu, net GND-2
- added copper zone on F.Cu, net GND-2
- added copper zone on B.Cu, net GND-3
- added copper zone on F.Cu, net GND-3
Other:
- board size 98.8 x 95.5 mm -> 98.8 x 94 mm

Commit message: 一旦完成
Parts:
- renumbered DPS311 to DPS310, J3 to URM37, J10 to pot
Other:
- outline, holes or cut-outs redrawn
- board text added: "A"
- board text added: "B"
- board text added: "RE12E"
- board text added: "←"

Commit message: edited boards
Parts:
- added R24: 220k, Resistor_SMD:R_0603_1608Metric_Pad0.98x0.95mm_HandSolder, B.Cu at (196.5, 45.5)
- added R28: 220k, Resistor_SMD:R_0603_1608Metric_Pad0.98x0.95mm_HandSolder, B.Cu at (196.5, 49.0)
- added R33: 220k, Resistor_SMD:R_0603_1608Metric_Pad0.98x0.95mm_HandSolder, F.Cu at (150.0, 113.5)
- added R34: 220k, Resistor_SMD:R_0603_1608Metric_Pad0.98x0.95mm_HandSolder, F.Cu at (152.1, 115.6)
- added R35: 220k, Resistor_SMD:R_0603_1608Metric_Pad0.98x0.95mm_HandSolder, B.Cu at (235.0, 89.5)
- added R36: 220k, Resistor_SMD:R_0603_1608Metric_Pad0.98x0.95mm_HandSolder, B.Cu at (238.0, 89.4)
- moved R2 0.55 mm to (177.5, 105.0)
- renumbered DPS310 to DPS311, pot to J10, URM37 to J3
Connections:
- R26 pad 1: +5V -> +3.3V-1
- R27 pad 1: +5V -> +3.3V-1
- U11 pad 3: /3. TFT/Pot_trim -> /3. TFT/V_check-3
- U5 pad 1: unconnected-(U5-GPIO2_A0_D0-Pad1) -> /2.logger/V_check-2
- U9 pad 14: +5V -> unconnected-(U9-5V-Pad14)
- U9 pad 2: unconnected-(U9-GPIO3_A1_D1-Pad2) -> /1. airdata/V_check-1
Routing:
- net +3.3V-3: track 205.1 -> 277.5 mm, vias 0 -> 1
- net +3.3V-2: track 92.9 -> 155.7 mm, vias 2 -> 5
- net +BATT-2: track 77.4 -> 120.5 mm
- net GND-3: track 54.9 -> 74.7 mm, vias 91 -> 33
- net +BATT-1: track 30.8 -> 46.7 mm
- net /3. TFT/V_check-3: track 0.00 -> 10.9 mm, vias 0 -> 1
- net +5V: track 10.4 -> 0.00 mm
- net +3.3V-1: track 74.9 -> 84.5 mm
- net /1. airdata/V_check-1: track 0.00 -> 8.71 mm, vias 0 -> 1
- net Net-(J11-Pin_2): track 4.98 -> 12.9 mm
- net GND-2: track 66.8 -> 74.1 mm, vias 4 -> 37
- net +BATT-3: track 36.9 -> 43.5 mm
- net /2.logger/V_check-2: track 0.00 -> 5.73 mm, vias 0 -> 2
- net /1. airdata/RS485_B: track 15.1 -> 13.4 mm
- net GND-1: track 177.1 -> 178.7 mm, vias 5 -> 31
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
Commit message: edited boards
Parts:
- added REF**: MountingHole_2.2mm_M2, MountingHole:MountingHole_2.2mm_M2, F.Cu at (219.0, 118.5)
- moved J11 1.07 mm to (230.0, 115.3)
Routing:
- net GND-1: track 178.7 -> 179.2 mm
